File: ProyectoTransversal.kicad_pcb (KiCad board)
At the start: 2 copper layers, 24 parts, among them J1 Conn_01x19, J2 Conn_01x19, J3 Screw_Terminal_01x02, J4 Screw_Terminal_01x02, J5 Conn_01x04, K1 Relay_SPDT, Q1 IRLZ44N, Q2 BC547, U1 DS18B20, U2 LM2596S-5

Commit message: Add R5 pull down cmd relay
Parts:
- added R5: 10k, Resistor_THT:R_Axial_DIN0207_L6.3mm_D2.5mm_P10.16mm_Horizontal, F.Cu at (187.1, 108.5)
Changed lines of the file:
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@@
+		)
+	)
+	(footprint "Resistor_THT:R_Axial_DIN0207_L6.3mm_D2.5mm_P10.16mm_Horizontal"
+		(layer "F.Cu")
+		(at 187.08 108.5 180)
+		(descr "Resistor, Axial_DIN0207 series, Axial, Horizontal, pin pitch=10.16mm, 0.25W = 1/4W, length*diameter=6.3*2.5mm^2, http://cdn-reichelt.de/documents/datenblatt/B400/1_4W%23YAG.pdf")
+		(tags "Resistor Axial_DIN0207 series Axial Horizontal pin pitch 10.16mm 0.25W = 1/4W length 6.3mm diameter 2.5mm")
+		(property "Reference" "R5"
+			(at 5.08 -2.37 0)
+			(layer "F.SilkS")
+			(effects
+				(font
+					(size 1 1)
+					(thickness 0.15)
+				)
+			)
+		)
+		(property "Value" "10k"
+			(at 5.08 2.37 0)
+			(layer "F.Fab")
+			(effects
+				(font
+					(size 1 1)
+					(thickness 0.15)
+				)
+			)
+		)
+		(property "Datasheet" ""
+			(at 0 0 0)
+			(layer "F.Fab")
+			(hide yes)
+			(effects
+				(font
+					(size 1.27 1.27)
+				)
+			)
+		)
+		(property "Description" "Resistor"
+			(at 0 0 0)
+			(layer "F.Fab")
+			(hide yes)
+			(effects
+				(font
+					(size 1.27 1.27)
+				)
+			)
+		)
+		(property "KiLib_Generator" "resistor/THT"
+			(at 0 0 0)
+			(layer "F.SilkS")
+			(hide yes)
+			(effects
+				(font
+					(size 1 1)
+					(thickness 0.15)
+				)
+			)
+		)
+		(property "Link" ""
+			(at 0 0 180)
+			(unlocked yes)
+			(layer "F.Fab")
+			(hide yes)
+			(effects
+				(font
+					(size 1 1)
+					(thickness 0.15)
+				)
+			)
+		)
+		(property ki_fp_filters "R_*")
+		(sheetname "/")
+		(sheetfile "ProyectoTransversal.kicad_sch")
+		(units
+			(unit
+				(name "A")
+				(pins "1" "2")
+			)
+		)
+		(attr through_hole)
+		(duplicate_pad_numbers_are_jumpers no)
+		(fp_line
+			(start 9.12 0)
+			(end 8.35 0)
+			(stroke
+				(width 0.12)
+				(type solid)
+			)
+			(layer "F.SilkS")
+		)
+		(fp_line
+			(start 1.04 0)
+			(end 1.81 0)
+			(stroke
+				(width 0.12)
+				(type solid)
+			)
+			(layer "F.SilkS")
+		)
+		(fp_rect
+			(start 1.81 -1.37)
+			(end 8.35 1.37)
+			(stroke
+				(width 0.12)
+				(type solid)
+			)
+			(fill no)
+			(layer "F.SilkS")
+		)
+		(fp_rect
+			(start -1.05 -1.5)
+			(end 11.21 1.5)
+			(stroke
+				(width 0.05)
+				(type solid)
+			)
+			(fill no)
+			(layer "F.CrtYd")
+		)
+		(fp_line
+			(start 10.16 0)
+			(end 8.23 0)
+			(stroke
+				(width 0.1)
+				(type solid)
+			)
+			(layer "F.Fab")
+		)
+		(fp_line
+			(start 0 0)
+			(end 1.93 0)
+			(stroke
+				(width 0.1)
+				(type solid)
+			)
+			(layer "F.Fab")
+		)
+		(fp_rect
+			(start 1.93 -1.25)
+			(end 8.23 1.25)
+			(stroke
+				(width 0.1)
+				(type solid)
+			)
+			(fill no)
+			(layer "F.Fab")
+		)
+		(fp_text user "${REFERENCE}"
+			(at 5.08 0 0)
+			(layer "F.Fab")
+			(effects
+				(font
+					(size 1 1)
+					(thickness 0.15)
+				)
+			)
+		)
+		(pad "1" thru_hole circle
+			(at 0 0 180)
+			(size 1.6 1.6)
+			(drill 0.8)
+			(layers "*.Cu" "*.Mask")
+			(remove_unused_layers no)
+			(net "/CMD_Relay")
+			(pintype "passive")
+		)
+		(pad "2" thru_hole circle
+			(at 10.16 0 180)
+			(size 1.6 1.6)
+			(drill 0.8)
+			(layers "*.Cu" "*.Mask")
+			(remove_unused_layers no)
+			(net "GND")
+			(pintype "passive")
+		)
+		(embedded_fonts no)
+		(model "${KICAD10_3DMODEL_DIR}/Resistor_THT.3dshapes/R_Axial_DIN0207_L6.3mm_D2.5mm_P10.16mm_Horizontal.step"
+			(offset
+				(xyz 0 0 0)
+			)
+			(scale
+				(xyz 1 1 1)
+			)
+			(rotate
+				(xyz 0 0 0)
+			)
 		)
 	)

Commit message: Begin reroute
Parts:
- moved R5 10.2 mm to (176.9, 108.5), turned to 0 degrees
- moved J5 5.24 mm to (149.0, 128.4)
- moved U1 4.92 mm to (156.0, 134.3), turned to 90 degrees
- moved R3 3.46 mm to (163.5, 127.7), turned to -90 degrees
Routing:
- net GND: track 43.1 -> 287.5 mm
- net /PWM_OUT: track 12.2 -> 78.6 mm
- net /SDA: track 0.00 -> 32.0 mm
- net /SCL: track 0.00 -> 23.4 mm
- net /CMD_Relay: track 0.00 -> 7.19 mm
- net /3V3: track 23.4 -> 27.5 mm
- net /sensor_temp: track 11.5 -> 9.49 mm

Commit message: Last changes to WIPM1U4
Parts:
- moved REF** 13.5 mm to (230.0, 143.5)
- moved D1 11.2 mm to (203.5, 94.5), turned to 180 degrees
- moved Q1 9.50 mm to (207.5, 131.1)
- moved REF** 3.64 mm to (127.5, 63.5)
- moved REF** 3.50 mm to (127.0, 143.5)
- moved C2 0.50 mm to (175.5, 84.0)
- moved REF** 0.50 mm to (230.0, 63.5)
Connections:
- J1 pad 10: unconnected-(J1-Pin_10-Pad10) -> /CMD_Relay
- J2 pad 7: /CMD_Relay -> unconnected-(J2-Pin_7-Pad7)
Routing:
- net /V_reg: track 39.8 -> 86.4 mm
- net /sensor_temp: track 9.49 -> 56.0 mm
- net Net-(D1-A): track 9.86 -> 35.8 mm
- net /CMD_Relay: track 7.19 -> 19.2 mm
- net Net-(J3-Pin_1): track 19.6 -> 10.6 mm
- net /GATE: track 13.0 -> 21.4 mm
- net GND: track 287.5 -> 292.9 mm
