File: ProyectoTransversal.kicad_sch (KiCad schematic)
At the start: 20 parts, among them J1 Conn_01x19, J2 Conn_01x19, J3 Screw_Terminal_01x02, J4 Screw_Terminal_01x02, J5 Conn_01x04, K1 Relay_SPDT, Q1 IRLZ44N, Q2 BC547, U1 DS18B20, U2 LM2596S-5

Commit message: Finish SCH layout
Parts:
- C1: value 220uF -> 100uF; footprint (none) -> Capacitor_THT:CP_Radial_D6.3mm_P2.50mm
- C2: value 100uF -> 220uF; footprint (none) -> Capacitor_THT:CP_Radial_D5.0mm_P2.50mm
- HS1: footprint (none) -> Heatsink:Heatsink_Fischer_SK104-STC-STIC_35x13mm_2xDrill2.5mm
- J1, J2, J5: footprint (none) -> Connector_PinHeader_2.54mm:PinHeader_1x19_P2.54mm_Vertical
- J3, J4: footprint (none) -> TerminalBlock:TerminalBlock_MaiXu_MX126-5.0-02P_1x02_P5.00mm
- K1: footprint (none) -> Relay_THT:Relay_SPDT_SANYOU_SRD_Series_Form_C
- L1: value L -> 33uH; footprint (none) -> Inductor_THT:L_Radial_D10.5mm_P5.00mm_Abacron_AISR-01
- R1, R2, R3, R4: footprint (none) -> Resistor_THT:R_Axial_DIN0207_L6.3mm_D2.5mm_P10.16mm_Horizontal
- U2: footprint Package_TO_SOT_SMD:TO-263-5_TabPin3 -> Package_TO_SOT_THT:TO-220-5_Vertical
Connections:
- net 12V: now also K1.3; no longer K1.11
- net Alim_12V: now also K1.5; no longer K1.14
- net V_reg: now also K1.1; no longer K1.A1
- net at D1.2 (A), Q2.1 (C): now also K1.2; no longer K1.A2
Changed lines of the file:
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@@
 			)
 		)
-		(property "Footprint" ""
+		(property "Footprint" "TerminalBlock:TerminalBlock_MaiXu_MX126-5.0-02P_1x02_P5.00mm"
 			(at 73.66 31.75 0)
 			(hide yes)
@@
 			)
 		)
-		(property "Footprint" "Package_TO_SOT_SMD:TO-263-5_TabPin3"
+		(property "Footprint" "Package_TO_SOT_THT:TO-220-5_Vertical"
 			(at 118.11 33.02 0)
 			(hide yes)
@@
 			)
 		)
-		(property "Footprint" ""
+		(property "Footprint" "Connector_PinHeader_2.54mm:PinHeader_1x19_P2.54mm_Vertical"
 			(at 254 106.68 0)
 			(hide yes)
@@
 			)
 		)
-		(property "Footprint" ""
+		(property "Footprint" "Resistor_THT:R_Axial_DIN0207_L6.3mm_D2.5mm_P10.16mm_Horizontal"
 			(at 224.282 133.35 90)
 			(hide yes)
@@
 			)
 		)
-		(property "Value" "100uF"
+		(property "Value" "220uF"
 			(at 153.67 35.9409 0)
 			(show_name no)
@@
 			)
 		)
-		(property "Footprint" ""
+		(property "Footprint" "Capacitor_THT:CP_Radial_D5.0mm_P2.50mm"
 			(at 150.8252 39.37 0)
 			(hide yes)
@@
 			)
 		)
-		(property "Footprint" ""
+		(property "Footprint" "Heatsink:Heatsink_Fischer_SK104-STC-STIC_35x13mm_2xDrill2.5mm"
 			(at 147.6248 105.41 0)
 			(hide yes)
@@
 			)
 		)
-		(property "Footprint" ""
+		(property "Footprint" "Connector_PinHeader_2.54mm:PinHeader_1x19_P2.54mm_Vertical"
 			(at 58.42 91.44 0)
 			(hide yes)
@@
 			)
 		)
-		(property "Footprint" ""
+		(property "Footprint" "Resistor_THT:R_Axial_DIN0207_L6.3mm_D2.5mm_P10.16mm_Horizontal"
 			(at 118.11 137.668 90)
 			(hide yes)
@@
 			)
 		)
-		(property "Footprint" ""
+		(property "Footprint" "TerminalBlock:TerminalBlock_MaiXu_MX126-5.0-02P_1x02_P5.00mm"
 			(at 139.7 119.38 0)
 			(hide yes)
@@
 			)
 		)
-		(property "Footprint" ""
+		(property "Footprint" "Resistor_THT:R_Axial_DIN0207_L6.3mm_D2.5mm_P10.16mm_Horizontal"
 			(at 246.38 85.598 90)
 			(hide yes)
@@
 			)
 		)
-		(property "Footprint" ""
+		(property "Footprint" "Connector_PinHeader_2.54mm:PinHeader_1x19_P2.54mm_Vertical"
 			(at 100.33 91.44 0)
 			(hide yes)
@@
 			)
 		)
-		(property "Value" "220uF"
+		(property "Value" "100uF"
 			(at 95.25 35.9409 0)
 			(show_name no)
@@
 			)
 		)
-		(property "Footprint" ""
+		(property "Footprint" "Capacitor_THT:CP_Radial_D6.3mm_P2.50mm"
 			(at 92.4052 39.37 0)
 			(hide yes)
@@
 			)
 		)
-		(property "Footprint" ""
+		(property "Footprint" "Relay_THT:Relay_SPDT_SANYOU_SRD_Series_Form_C"
 			(at 179.07 69.85 0)
 			(hide yes)
@@
 			)
 		)
-		(pin "A2"
-		)
-		(pin "A1"
-		)
-		(pin "14"
-		)
-		(pin "11"
-		)
-		(pin "12"
+		(pin "5"
+		)
+		(pin "1"
+		)
+		(pin "3"
+		)
+		(pin "2"
+		)
+		(pin "4"
 		)
 		(instances
@@
 			)
 		)
-		(property "Footprint" ""
+		(property "Footprint" "Resistor_THT:R_Axial_DIN0207_L6.3mm_D2.5mm_P10.16mm_Horizontal"
 			(at 104.902 142.24 90)
 			(hide yes)
@@
 			)
 		)
-		(property "Value" "L"
+		(property "Value" "33uH"
 			(at 145.542 26.67 90)
 			(show_name no)
@@
 			)
 		)
-		(property "Footprint" ""
+		(property "Footprint" "Inductor_THT:L_Radial_D10.5mm_P5.00mm_Abacron_AISR-01"
 			(at 143.51 29.21 0)
 			(hide yes)

Commit message: Route voltage regulator
Parts:
- J5: footprint Connector_PinHeader_2.54mm:PinHeader_1x19_P2.54mm_Vertical -> Connector_PinHeader_2.54mm:PinHeader_1x04_P2.54mm_Vertical
Changed lines of the file:
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@@
 			)
 		)
-		(property "Footprint" "Connector_PinHeader_2.54mm:PinHeader_1x19_P2.54mm_Vertical"
+		(property "Footprint" "Connector_PinHeader_2.54mm:PinHeader_1x04_P2.54mm_Vertical"
 			(at 254 106.68 0)
 			(hide yes)
@@
 		)
 		(property "Value" "1k"
-			(at 245.11 78.74 90)
-			(show_name no)
-			(do_not_autoplace no)
+			(at 249.682 81.28 90)
+			(show_name no)
+			(do_not_autoplace no)

Commit message: Add R5 pull down cmd relay
Parts:
- added R5: 10k, Resistor_THT:R_Axial_DIN0207_L6.3mm_D2.5mm_P10.16mm_Horizontal, symbol Device:R
Connections:
- net CMD_Relay: now also R5.1
- net GND: now also R5.2
Other:
- moved on the sheet: J5, R4

Commit message: Last changes to WIPM1U4
Connections:
- net CMD_Relay: now also J1.10 (Pin_10); no longer J2.7 (Pin_7)
Changed lines of the file:
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@@
 	(wire
 		(pts
-			(xy 45.72 83.82) (xy 53.34 83.82)
-		)
-		(stroke
-			(width 0)
-			(type default)
-		)
-	)
-	(wire
-		(pts
 			(xy 91.44 24.13) (xy 91.44 31.75)
 		)
@@
 	(wire
 		(pts
+			(xy 85.09 91.44) (xy 95.25 91.44)
+		)
+		(stroke
+			(width 0)
+			(type default)
+		)
+	)
+	(wire
+		(pts
 			(xy 116.84 34.29) (xy 116.84 41.91)
 		)
@@
 	)
 	(label "CMD_Relay"
-		(at 45.72 83.82 0)
+		(at 85.09 91.44 0)
 		(effects
 			(font
