File: _restore_backup_2026-08-05T16-04-41-681/ProyectoTransversal.kicad_sch (KiCad schematic)
At the start: 21 parts, among them J1 Conn_01x19, J2 Conn_01x19, J3 Screw_Terminal_01x02, J4 Screw_Terminal_01x02, J5 Conn_01x04, K1 Relay_SPDT, Q1 IRLZ44N, Q2 BC547, U1 DS18B20, U2 LM2596S-5

Commit message: Final submission
Parts:
- C1, C2, R1, R2, R3, R4, R5: Tecnologia SMD -> (none)
- D1, D2, HS1, J1, J2, J3, J4, J5, K1, L1, Q1, Q2, U1, U2: Tecnologia THT -> (none)
Changed lines of the file:
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@@
 			)
 		)
-		(property "KiLib_Generator" "terminal_block/MaiXu"
+		(property "Link" ""
 			(at 73.66 31.75 0)
 			(hide yes)
@@
 			)
 		)
-		(property "Tecnologia" "THT"
+		(property "KiLib_Generator" "terminal_block/MaiXu"
 			(at 73.66 31.75 0)
 			(hide yes)
@@
 			)
 		)
-		(property "Tecnologia" "THT"
+		(property "Link" ""
 			(at 210.82 139.7 0)
 			(hide yes)
@@
 			)
 		)
-		(property "KiLib_Generator" "package/TO_SOT/THT"
+		(property "Link" ""
 			(at 116.84 26.67 0)
 			(hide yes)
@@
 			)
 		)
-		(property "Tecnologia" "THT"
+		(property "KiLib_Generator" "package/TO_SOT/THT"
 			(at 116.84 26.67 0)
 			(hide yes)
@@
 			)
 		)
-		(property "KiLib_Generator" "connector/pin_header_socket"
+		(property "Link" ""
 			(at 255.27 110.49 0)
 			(hide yes)
@@
 			)
 		)
-		(property "Tecnologia" "THT"
+		(property "KiLib_Generator" "connector/pin_header_socket"
 			(at 255.27 110.49 0)
 			(hide yes)
@@
 			)
 		)
-		(property "KiLib_Generator" "SMD_2terminal_chip_molded"
+		(property "Link" ""
 			(at 226.06 133.35 0)
 			(hide yes)
@@
 			)
 		)
-		(property "Tecnologia" "SMD"
+		(property "KiLib_Generator" "SMD_2terminal_chip_molded"
 			(at 226.06 133.35 0)
 			(hide yes)
@@
 			)
 		)
-		(property "KiLib_Generator" "capacitor/SMD/elec_round_polarized"
+		(property "Link" ""
 			(at 149.86 35.56 0)
 			(hide yes)
@@
 			)
 		)
-		(property "Tecnologia" "SMD"
+		(property "KiLib_Generator" "capacitor/SMD/elec_round_polarized"
 			(at 149.86 35.56 0)
 			(hide yes)
@@
 			)
 		)
-		(property "KiLib_Generator" "diode/THT"
-			(at 223.52 68.58 0)
+		(property "Link" ""
+			(at 223.52 68.58 90)
 			(hide yes)
 			(show_name no)
@@
 			)
 		)
-		(property "Tecnologia" "THT"
-			(at 223.52 68.58 90)
+		(property "KiLib_Generator" "diode/THT"
+			(at 223.52 68.58 0)
 			(hide yes)
 			(show_name no)
@@
 			)
 		)
-		(property "Tecnologia" "THT"
+		(property "Link" ""
 			(at 147.32 105.41 0)
 			(hide yes)
@@
 			)
 		)
-		(property "KiLib_Generator" "package/TO_SOT/THT"
+		(property "Link" ""
 			(at 137.16 135.89 0)
 			(hide yes)
@@
 			)
 		)
-		(property "Tecnologia" "THT"
+		(property "KiLib_Generator" "package/TO_SOT/THT"
 			(at 137.16 135.89 0)
 			(hide yes)
@@
 			)
 		)
-		(property "KiLib_Generator" "connector/pin_header_socket"
+		(property "Link" ""
 			(at 58.42 91.44 0)
 			(hide yes)
@@
 			)
 		)
-		(property "Tecnologia" "THT"
+		(property "KiLib_Generator" "connector/pin_header_socket"
 			(at 58.42 91.44 0)
 			(hide yes)
@@
 			)
 		)
-		(property "KiLib_Generator" "SMD_2terminal_chip_molded"
-			(at 118.11 135.89 0)
+		(property "Link" ""
+			(at 118.11 135.89 90)
 			(hide yes)
 			(show_name no)
@@
 			)
 		)
-		(property "Tecnologia" "SMD"
-			(at 118.11 135.89 90)
+		(property "KiLib_Generator" "SMD_2terminal_chip_molded"
+			(at 118.11 135.89 0)
 			(hide yes)
 			(show_name no)
@@
 			)
 		)
-		(property "KiLib_Generator" "diode/THT"
+		(property "Link" ""
 			(at 128.27 41.91 0)
 			(hide yes)
@@
 			)
 		)
-		(property "Tecnologia" "THT"
+		(property "KiLib_Generator" "diode/THT"
 			(at 128.27 41.91 0)
 			(hide yes)
@@
 			)
 		)
-		(property "KiLib_Generator" "terminal_block/MaiXu"
-			(at 139.7 119.38 0)
+		(property "Link" ""
+			(at 139.7 119.38 90)
 			(hide yes)
 			(show_name no)
@@
 			)
 		)
-		(property "Tecnologia" "THT"
-			(at 139.7 119.38 90)
+		(property "KiLib_Generator" "terminal_block/MaiXu"
+			(at 139.7 119.38 0)
 			(hide yes)
 			(show_name no)
@@
 			)
 		)
-		(property "Tecnologia" "THT"
+		(property "Link" ""
 			(at 226.06 83.82 0)
 			(hide yes)
@@
 			)
 		)
-		(property "KiLib_Generator" "SMD_2terminal_chip_molded"
-			(at 238.76 83.82 0)
+		(property "Link" ""
+			(at 238.76 83.82 90)
 			(hide yes)
 			(show_name no)
@@
 			)
 		)
-		(property "Tecnologia" "SMD"
-			(at 238.76 83.82 90)
+		(property "KiLib_Generator" "SMD_2terminal_chip_molded"
+			(at 238.76 83.82 0)
 			(hide yes)
 			(show_name no)
@@
 			)
 		)
-		(property "KiLib_Generator" "connector/pin_header_socket"
+		(property "Link" ""
 			(at 100.33 91.44 0)
 			(hide yes)
@@
 			)
 		)
-		(property "Tecnologia" "THT"
+		(property "KiLib_Generator" "connector/pin_header_socket"
 			(at 100.33 91.44 0)
 			(hide yes)
@@
 			)
 		)
-		(property "KiLib_Generator" "capacitor/SMD/elec_round_polarized"
+		(property "Link" ""
 			(at 91.44 35.56 0)
 			(hide yes)
@@
 			)
 		)
-		(property "Tecnologia" "SMD"
+		(property "KiLib_Generator" "capacitor/SMD/elec_round_polarized"
 			(at 91.44 35.56 0)
 			(hide yes)
@@
 			)
 		)
-		(property "Tecnologia" "THT"
+		(property "Link" ""
 			(at 190.5 68.58 0)
 			(hide yes)
@@
 			)
 		)
-		(property "KiLib_Generator" "SMD_2terminal_chip_molded"
+		(property "Link" ""
 			(at 106.68 142.24 0)
 			(hide yes)
@@
 			)
 		)
-		(property "Tecnologia" "SMD"
+		(property "KiLib_Generator" "SMD_2terminal_chip_molded"
 			(at 106.68 142.24 0)
 			(hide yes)
@@
 			)
 		)
-		(property "KiLib_Generator" "SMD_2terminal_chip_molded"
+		(property "Link" ""
 			(at 247.65 88.9 0)
 			(hide yes)
@@
 			)
 		)
-		(property "Tecnologia" "SMD"
+		(property "KiLib_Generator" "SMD_2terminal_chip_molded"
 			(at 247.65 88.9 0)
 			(hide yes)
@@
 			)
 		)
-		(property "KiLib_Generator" "choke_THT"
-			(at 143.51 29.21 0)
+		(property "Link" ""
+			(at 143.51 29.21 90)
 			(hide yes)
 			(show_name no)
@@
 			)
 		)
-		(property "Tecnologia" "THT"
-			(at 143.51 29.21 90)
+		(property "KiLib_Generator" "choke_THT"
+			(at 143.51 29.21 0)
 			(hide yes)
 			(show_name no)
